File: PCB/Modules/v0.7/Analog Output 4ch/AnalogOutputModule_4ch.sch (EAGLE design)
At the start: 40 parts, among them IC1 SN65HVD31DR, IC2 SN65HVD31DR, IC3 AD5754RBREZ, IC4 REF193GSZ

Commit message: -Improved Analog Output Module schematic organization and labeling -Thickened trace connecting Analog Output Module ground planes
Connections:
- net N$20 renamed REF_ENABLE
Other:
- note added: "3V Reference IC"
- note added: "DC Converter + AD5754R DAC"
- note added: "Ground plane bridge"
- note added: "NOTE: This design file is part of the Sanworks Bpod repository. (C) 2017 Sanworks LLC"
- note added: "Please read GPL v3.0 for license terms. http//www.gnu.org/licenses/gpl-3.0.en.html"
- note added: "REF_ENABLE"
- note added: "Sanworks LLC"
- note added: "Teensy 3.6 + RS-485 Interface"
- note added: "http://github.com/sanworks/Bpod"
- moved on the sheet: AGND, BNC1, BNC2, BNC3, BNC4, C10, C11, C12, C13, C14, C15, C3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
