File: PCB/Modules/v0.7/Valve Driver Module/ValveModule_r1.brd (EAGLE design)
At the start: 40.2 x 83 mm, 23 parts, among them IC1 SN65HVD31DR, IC2 LM3480-5.0, IC3 ISO1H811G, J8 POWER_JACK

Commit message: -Updated silk screen, improved trace clearance and reorganized schematic for ValveModule PCB
Parts:
- renumbered U$1 to J10
Routing:
- net GNDBB: track 9.29 -> 18.2 mm
Other:
- board text added: "IC3"
- board text added: "J10"
