File: PCB/Modules/v0.7/Valve Driver Module/ValveModule_r1.sch (EAGLE design)
At the start: 23 parts, among them IC1 SN65HVD31DR, IC2 LM3480-5.0, IC3 ISO1H811G, J8 POWER_JACK

Commit message: -Updated silk screen, improved trace clearance and reorganized schematic for ValveModule PCB
Parts:
- removed U$1: RJ45-8PTH, SparkFun:RJ45-8PTH
- added J10: RJ45-8PTH, SparkFun:RJ45-8PTH
Connections:
- net GND: now also J10.6; no longer U$1.6
- net N$10: now also J10.4; no longer U$1.4
- net N$24: now also J10.5; no longer U$1.5
- net N$7: now also J10.1; no longer U$1.1
- net N$8: now also J10.2; no longer U$1.2
- net N$9: now also J10.3; no longer U$1.3
Other:
- note added: "Isolated valve driver IC"
- note added: "NOTE: This design file is part of the Sanworks Bpod repository. (C) 2016 Sanworks LLC"
- note added: "Please read GPL v3.0 for license terms. http//www.gnu.org/licenses/gpl-3.0.en.html"
- note added: "Sanworks LLC"
- note added: "UART/RS485 and MCU power interface"
- note added: "http://github.com/sanworks/Bpod"
- moved on the sheet: C1, C2, C3, C4, C5, D1, H1, H2, H3, H4, IC1, IC2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

Commit message: -Added SNES Module PCB design -Added SNES Module bottom-guard design -Added DDS Module enclosure -Updated link to Bpod-CAD repository in schematic files
Other:
- note added: "NOTE: This design file is part of the Sanworks Bpod-CAD repository. (C) 2016 Sanworks LLC"
- note added: "http://github.com/sanworks/Bpod-CAD"
- note removed: "NOTE: This design file is part of the Sanworks Bpod repository. (C) 2016 Sanworks LLC"
- note removed: "http://github.com/sanworks/Bpod"
Changed lines of the file:
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@@
 <text x="25.4" y="228.6" size="5.08" layer="94" font="vector">UART/RS485 and MCU power interface</text>
 <text x="238.76" y="228.6" size="5.08" layer="94" font="vector">Isolated valve driver IC</text>
-<text x="28.448" y="24.384" size="5.08" layer="94" font="vector">Please read GPL v3.0 for license terms. http//www.gnu.org/licenses/gpl-3.0.en.html</text>
-<text x="1.778" y="34.29" size="5.08" layer="94" font="vector">NOTE: This design file is part of the Sanworks Bpod repository. (C) 2016 Sanworks LLC</text>
+<text x="28.448" y="24.384" size="3.81" layer="94" font="vector">Please read GPL v3.0 for license terms. http//www.gnu.org/licenses/gpl-3.0.en.html</text>
+<text x="1.778" y="34.29" size="3.81" layer="94" font="vector">NOTE: This design file is part of the Sanworks Bpod-CAD repository. (C) 2016 Sanworks LLC</text>
 <wire x1="203.2" y1="119.38" x2="375.92" y2="119.38" width="1.016" layer="94" style="longdash"/>
 <text x="284.48" y="8.89" size="3.81" layer="94" font="vector">Sanworks LLC</text>
-<text x="1.778" y="1.016" size="5.08" layer="94" font="vector">http://github.com/sanworks/Bpod</text>
+<text x="1.778" y="1.016" size="5.08" layer="94" font="vector">http://github.com/sanworks/Bpod-CAD</text>
 </plain>
 <instances>
