File: PCB/BpodStateMachine/r0.8/BpodMainBoard_r0_8.sch (EAGLE design)
At the start: 54 parts, among them IC1 OPTOISOLATOR-2SOIC8, IC10 ADUM5240, IC2 CD4050, IC3 OPTOISOLATOR-2SOIC8, IC4 CD4050, IC5 SN65HVD31DR, IC7 CY15B104Q-SXI, IC8 SN65HVD31DR, IC9 SN65HVD31DR

Commit message: -Added SNES Module PCB design -Added SNES Module bottom-guard design -Added DDS Module enclosure -Updated link to Bpod-CAD repository in schematic files
Other:
- note added: "NOTE: This design file is part of the Sanworks Bpod-CAD repository. (C) 2017 Sanworks LLC"
- note added: "http://github.com/sanworks/Bpod-CAD"
- note removed: "NOTE: This design file is part of the Sanworks Bpod repository. (C) 2016 Sanworks LLC"
- note removed: "http://github.com/sanworks/Bpod"
Changed lines of the file:
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@@
 <wire x1="-147.574" y1="-1.524" x2="-22.86" y2="-1.524" width="0.1524" layer="94" style="longdash"/>
 <text x="-258.572" y="-117.856" size="5.08" layer="94" font="vector">Please read GPL v3.0 for license terms. http//www.gnu.org/licenses/gpl-3.0.en.html</text>
-<text x="-285.242" y="-107.95" size="5.08" layer="94" font="vector">NOTE: This design file is part of the Sanworks Bpod repository. (C) 2016 Sanworks LLC</text>
+<text x="-285.242" y="-107.95" size="5.08" layer="94" font="vector">NOTE: This design file is part of the Sanworks Bpod-CAD repository. (C) 2017 Sanworks LLC</text>
 <text x="-279.908" y="-13.208" size="5.08" layer="94" font="vector">Wire Terminals / Optoisolator</text>
 <wire x1="-22.86" y1="-1.524" x2="-22.86" y2="66.04" width="0.1524" layer="94" style="longdash"/>
@@
 <text x="217.932" y="145.796" size="1.778" layer="95" rot="R270">LED_Red</text>
 <text x="200.152" y="172.212" size="1.778" layer="95" rot="R270">LED_Green</text>
-<text x="19.558" y="-197.104" size="5.08" layer="94" font="vector">http://github.com/sanworks/Bpod</text>
+<text x="1.778" y="-192.024" size="5.08" layer="94" font="vector">http://github.com/sanworks/Bpod-CAD</text>
 <text x="234.95" y="-101.854" size="5.08" layer="94" font="vector">Holes</text>
 <text x="-134.62" y="-27.686" size="1.778" layer="95" rot="R180">Upper 5V</text>
