File: PCB/Modules/Gen2/Valve Driver Module/ValveModule_r2.brd (EAGLE design)
At the start: 40.2 x 83 mm, 23 parts, among them IC1 SN65HVD31DR, IC2 LM3480-5.0, IC3 ISO1H811G, J10 RJ45-8PTH, J8 POWER_JACK

Commit message: -Critical Update for modules with optional RJ45 power (ValveDriver, I2C, SNES and DDS); new PCB designs add a diode to prevent USB power from entering output pin of 5V regulator, when RJ45 (state machine) power is not connected. This update greatly reduces unnecessary power consumption and heat dissipation. If you built a board using the previous designs, please Email a photo of your board to Sanworks support for a free upgrade. -Updated component names on some boards and on web BOMs to avoid skipping parts -Renamed Gen2 module PCB folder from '0.7' to 'Gen2' -Retired pocket state machine (to be replaced with Bpod State Machine r1)
Parts:
- added D2: MBR0520LT, diode:SOD123
- moved J9 12.5 mm to (18.7, 20.6), turned to 180 degrees
Connections:
- new net N$25: C4.2, IC2.1, J9.1
- net 5V: now also D2.C; no longer C4.2, IC2.1
- net N$24: now also C5.2, IC2.2; no longer J9.2
- net N$26: now also D2.A, J9.2; no longer C5.2, IC2.2, J9.1
Routing:
- net 5V: track 39.5 -> 24.0 mm
- net N$24: track 17.1 -> 26.8 mm, vias 0 -> 1
- net N$25: track 0.00 -> 6.67 mm
- net N$26: track 7.47 -> 2.65 mm
- net GND: track 51.8 -> 52.8 mm
Other:
- board text added: "+"
- board text added: "Module r2"
- board text added: "PWR"
- board text removed: "Module r1"
- board text removed: "Power"
Changed lines of the file:
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@@
 <text x="7.0335" y="4.91" size="1.27" layer="21" font="vector" rot="R90">GND</text>
 <text x="32.497" y="42.655" size="1.5" layer="21" font="vector" rot="R270">Bpod Valve Driver</text>
-<text x="34.4865" y="42.722" size="1.5" layer="21" font="vector" rot="R270">Module r1</text>
+<text x="34.4865" y="42.722" size="1.5" layer="21" font="vector" rot="R270">Module r2</text>
 <text x="-2.456" y="69.997" size="1.5" layer="21" font="vector">1+</text>
 <text x="-2.3925" y="66.568" size="1.5" layer="21" font="vector">1-</text>
@@
 <text x="22.8165" y="81.704" size="1.5" layer="21" font="vector" rot="R270">12-24VDC</text>
 <text x="24.7215" y="81.637" size="1.5" layer="21" font="vector" rot="R270">Pos. Ctr</text>
-<text x="32.9795" y="16.8635" size="1.5" layer="21" font="vector" rot="R270">Power</text>
-<text x="31.0285" y="15.7415" size="1.5" layer="21" font="vector" rot="R270">Bpod</text>
+<text x="15.7765" y="15.6395" size="1.5" layer="21" font="vector">PWR</text>
+<text x="14.1385" y="17.5885" size="1.5" layer="21" font="vector">Bpod</text>
 <polygon width="1" layer="42">
 <vertex x="17.4" y="22.8"/>
@@
 <text x="25.197" y="8.881" size="1.27" layer="21" font="vector" rot="R270">J10</text>
 <text x="23.459" y="45.117" size="1.27" layer="21" font="vector">IC3</text>
+<text x="11.7" y="19.92" size="1" layer="21">+</text>
 </plain>
 <attributes>
@@
 <param name="mdPadPad" value="12mil"/>
 <param name="mdPadVia" value="12mil"/>
-<param name="mdViaVia" value="12mil"/>
+<param name="mdViaVia" value="6mil"/>
 <param name="mdSmdPad" value="0mil"/>
 <param name="mdSmdVia" value="0mil"/>
@@
 <attribute name="VALUE" x="11.711" y="64.604" size="1.27" layer="27" ratio="10"/>
 </element>
-<element name="J9" library="SparkFun-Connectors" package="1X02" value="" x="29.5275" y="14.2875" smashed="yes" rot="R270">
-<attribute name="NAME" x="28.7225" y="8.9645" size="1.016" layer="25" font="vector" ratio="10"/>
-<attribute name="VALUE" x="27.4955" y="15.5575" size="0.6096" layer="27" font="vector" ratio="20" rot="R270"/>
+<element name="J9" library="SparkFun-Connectors" package="1X02" value="" x="18.7275" y="20.6325" smashed="yes" rot="R180">
+<attribute name="NAME" x="17.7425" y="22.2245" size="1.016" layer="25" font="vector" ratio="10"/>
+<attribute name="VALUE" x="19.9975" y="22.6645" size="0.6096" layer="27" font="vector" ratio="20" rot="R180"/>
 </element>
 <element name="IC2" library="regulators" package="SOT-23-3" value="LM3480-5.0" x="25.9715" y="20.574" smashed="yes">
@@
 <element name="C3" library="JoshParts10" package="EEE-FK1H100UR" value="EEE-FK1H100UR" x="8.7" y="80.58" smashed="yes" rot="R180">
 <attribute name="NAME" x="7.86" y="73.89" size="1" layer="25" font="vector"/>
+</element>
+<element name="D2" library="diode" package="SOD123" value="MBR0520LT" x="13.56" y="22.26" smashed="yes" rot="R270">
+<attribute name="NAME" x="11.5" y="23.84" size="1" layer="25" font="vector" rot="R270"/>
 </element>
 </elements>
@@
 <wire x1="26.292" y1="21.847" x2="25.9715" y2="21.844" width="1" layer="1"/>
 <wire x1="22.482" y1="21.9075" x2="22.606" y2="22.101" width="1" layer="1"/>
-<wire x1="22.482" y1="21.9075" x2="22.1895" y2="22.2" width="1" layer="1"/>
-<wire x1="22.1895" y1="22.2" x2="15.6" y2="22.2" width="1" layer="1"/>
-<via x="15.6" y="22.2" extent="1-16" drill="0.8"/>
-<wire x1="15.6" y1="22.2" x2="15.6" y2="22.8" width="1" layer="16"/>
+<via x="15.54" y="23.7" extent="1-16" drill="0.8"/>
+<wire x1="15.54" y1="23.7" x2="15.6" y2="22.8" width="1" layer="16"/>
 <wire x1="22.606" y1="22.101" x2="22.863" y2="21.844" width="1" layer="1"/>
 <wire x1="22.863" y1="21.844" x2="25.9715" y2="21.844" width="1" layer="1"/>
+<wire x1="22.482" y1="21.9075" x2="21.5295" y2="22.86" width="1" layer="1"/>
+<wire x1="21.5295" y1="22.86" x2="16.38" y2="22.86" width="1" layer="1"/>
+<wire x1="16.38" y1="22.86" x2="15.54" y2="23.7" width="1" layer="1"/>
 </signal>
 <signal name="N$4">
@@
 <signal name="5V">
 <contactref element="J3" pad="1"/>
-<contactref element="IC2" pad="1"/>
-<contactref element="C4" pad="2"/>
-<wire x1="25.019" y1="19.304" x2="22.609" y2="19.304" width="1" layer="1"/>
-<wire x1="22.609" y1="19.304" x2="22.606" y2="19.301" width="1" layer="1"/>
-<wire x1="22.609" y1="19.304" x2="21.2725" y2="19.304" width="1" layer="1"/>
-<wire x1="21.2725" y1="19.304" x2="20.0025" y2="20.5105" width="1" layer="1"/>
-<wire x1="20.0025" y1="20.5105" x2="13.5255" y2="20.5105" width="1" layer="1"/>
-<wire x1="13.5255" y1="20.5105" x2="13.462" y2="29.9085" width="1" layer="1"/>
 <via x="13.462" y="29.9085" extent="1-16" drill="0.6"/>
 <wire x1="13.462" y1="29.9085" x2="9.9695" y2="29.9085" width="1" layer="16"/>
@@
 <wire x1="9.9695" y1="29.845" x2="2.032" y2="36.195" width="1" layer="1"/>
 <wire x1="2.032" y1="36.195" x2="2.032" y2="40.64" width="1" layer="1"/>
+<wire x1="13.462" y1="29.9085" x2="13.5" y2="29.8705" width="1" layer="1"/>
+<contactref element="D2" pad="C"/>
+<wire x1="13.56" y1="24.16" x2="13.62" y2="24.24" width="1" layer="1"/>
+<wire x1="13.62" y1="24.24" x2="13.44" y2="24.96" width="1" layer="1"/>
+<wire x1="13.44" y1="24.96" x2="13.44" y2="29.8865" width="1" layer="1"/>
+<wire x1="13.44" y1="29.8865" x2="13.462" y2="29.9085" width="1" layer="1"/>
 </signal>
 <signal name="N$2">
@@
 <signal name="N$24">
 <contactref element="J10" pad="5"/>
-<contactref element="J9" pad="2"/>
 <wire x1="17.526" y1="9.397" x2="17.526" y2="6.2865" width="1" layer="16"/>
 <wire x1="17.526" y1="6.2865" x2="23.114" y2="6.2865" width="1" layer="16"/>
-<wire x1="23.114" y1="6.2865" x2="29.5275" y2="11.7475" width="1" layer="16"/>
-</signal>
-<signal name="N$26">
-<contactref element="J9" pad="1"/>
 <contactref element="IC2" pad="2"/>
 <contactref element="C5" pad="2"/>
-<wire x1="29.5275" y1="14.2875" x2="29.5275" y2="19.047" width="1" layer="1"/>
 <wire x1="29.5275" y1="19.047" x2="27.181" y2="19.047" width="1" layer="1"/>
 <wire x1="27.181" y1="19.047" x2="26.924" y2="19.304" width="1" layer="1"/>
+<wire x1="23.114" y1="6.2865" x2="29.52" y2="12.6925" width="1" layer="16"/>
+<wire x1="29.52" y1="12.6925" x2="29.52" y2="14.76" width="1" layer="16"/>
+<via x="29.52" y="14.76" extent="1-16" drill="0.6"/>
+<wire x1="29.52" y1="14.76" x2="29.5275" y2="14.7675" width="1" layer="1"/>
+<wire x1="29.5275" y1="14.7675" x2="29.5275" y2="19.047" width="1" layer="1"/>
+</signal>
+<signal name="N$25">
+<contactref element="IC2" pad="1"/>
+<contactref element="C4" pad="2"/>
+<contactref element="J9" pad="1"/>
+<wire x1="18.7275" y1="20.6325" x2="21" y2="19.26" width="1" layer="1"/>
+<wire x1="21" y1="19.26" x2="22.606" y2="19.301" width="1" layer="1"/>
+<wire x1="22.606" y1="19.301" x2="25.019" y2="19.304" width="1" layer="1"/>
+</signal>
+<signal name="N$26">
+<contactref element="J9" pad="2"/>
+<contactref element="D2" pad="A"/>
+<wire x1="16.1875" y1="20.6325" x2="14.7525" y2="20.4525" width="1" layer="1"/>
+<wire x1="14.7525" y1="20.4525" x2="14.22" y2="20.4" width="1" layer="1"/>
+<wire x1="14.22" y1="20.4" x2="13.76" y2="20.34" width="1" layer="1"/>
+<wire x1="13.76" y1="20.34" x2="13.56" y2="20.36" width="1" layer="1"/>
 </signal>
 </signals>
