File: PCB/BpodStateMachine/r2.1/BpodFSM_r2_1.sch (EAGLE design)
At the start: 44 parts, among them IC1 SN65HVD31DR, IC10 MTU1D0505MC, IC11 MTU1D0505MC, IC2 SN65HVD31DR, IC3 SN65HVD31DR, IC4 SN65HVD31DR, IC5 SN65HVD31DR, IC6 OPTOISOLATOR-2SOIC8, IC7 ADUM5240, IC9 MTU1D0505MC

Commit message: -Updated PCB designs for all boards with Teensy 3.5 + 3.6 to optimize solder pads for assembly (new designs validated 12 JAN 2018). No components changed. -Optimized silk screens on PCBs above to ensure that each component name is clearly visible (previously overlapped with vias in some cases) -Improved design of Bpod 2 enclosure for added mechanical strength
Parts:
- added C11, C12, C13: 0.1uf, SparkFun-Capacitors:CAP1206
- added C14: EEE-FK1H100UR, JoshParts10:EEE-FK1H100UR
- added D1: (no value), diode:DIODE-DO214AA
- added IC12: CD4050, SparkFun-DigitalIC:CD4050
- added IC8: ISO1H811G, JoshParts10:ISO1H811G
- added J4: POWER_JACKSLT, SparkFun-Connectors:POWER_JACKSLT
- added PORT1, PORT2, PORT3, PORT4: RJ45-8PTH, SparkFun:RJ45-8PTH
- R2, R3: value 220 -> 1K
Connections:
- new net BNCOUT1: IC7.VI_B, U$1.4/CAN0-RX/SDA2/PWM
- new net BNCOUT2: IC7.VI_A, U$1.3/CAN0-TX/SCL2/PWM
- new net DRVR_ENBL: IC8.P$3, U$1.19/A5/T/SCL0
- new net GNDBB: C14.CATHODE, D1.A, IC8.P$19, J4.GND, J4.GNDBREAK, PORT1.7, PORT2.7, PORT3.7, PORT4.7
- new net N$31: IC12.5IN, PORT4.1
- new net N$56: IC12.2IN, PORT1.1
- new net PORT1IN: IC12.2OUT, U$1.39/A20
- new net PORT1LED: PORT1.3, U$1.37/A18/SCL1/PWM
- new net PORT2IN: IC12.3OUT, U$1.38/A19/SDA1/PWM
- new net PORT2LED: PORT2.3, U$1.14/A0/PWM
- new net PORT3IN: IC12.4OUT, U$1.18/A4/T/SDA0
- new net PORT3LED: PORT3.3, U$1.16/A2/T/PWM
- new net PORT4IN: IC12.5OUT, U$1.15/A1/T
- new net PORT4LED: PORT4.3, U$1.17/A3/T/PWM
- new net VBB: C14.ANODE, D1.C, IC8.VBB, J4.PWR
- new net VLV1IN: IC8.P$6, IC8.P$7, U$1.23/A9/T/PWM
- new net VLV1OUT: IC8.P$33, IC8.P$34, IC8.P$35, IC8.P$36, PORT1.6
- new net VLV2IN: IC8.P$8, IC8.P$9, U$1.22/A8/T/PWM
- new net VLV2OUT: IC8.P$29, IC8.P$30, IC8.P$31, IC8.P$32, PORT2.6
- new net VLV3IN: IC8.P$12, IC8.P$13, U$1.20/A6/PWM
- new net VLV3OUT: IC8.P$21, IC8.P$22, IC8.P$23, IC8.P$24, PORT3.6
- new net VLV4IN: IC8.P$10, IC8.P$11, U$1.21/A7/PWM
- new net VLV4OUT: IC8.P$25, IC8.P$26, IC8.P$27, IC8.P$28, PORT4.6
- net 5V: now also PORT1.4, PORT2.4, PORT3.4, PORT4.4
- net BNCIN1: now also U$1.6/PWM; no longer U$1.16/A2/T/PWM
- net BNCIN2: now also U$1.5/PWM; no longer U$1.17/A3/T/PWM
- net GND: now also C11.2, C12.1, C13.2, IC12.VSS, IC8.P$15, IC8.P$4, IC8.P$5, PORT1.5, PORT2.5, PORT3.5, PORT4.5
- net LED_GREEN: now also U$1.2/PWM; no longer U$1.30/T/PWM
- net LED_RED: now also U$1.36/A17/PWM; no longer U$1.29/T/PWM
- net N$20: now also IC12.3IN, PORT2.1; no longer IC7.VI_B, U$1.36/A17/PWM
- net N$24: now also IC12.4IN, PORT3.1; no longer IC7.VI_A, U$1.37/A18/SCL1/PWM
- net VCC: now also C11.1, C12.2, C13.1, IC12.VCC, IC8.P$2
Other:
- note added: "BNC input channels + optoisolator"
- note added: "BNC outputs + isolated driver"
- note added: "BNCOUT1"
- note added: "BNCOUT2"
- note added: "Behavior ports + logic level converter"
- note added: "DRVR_ENBL"
- note added: "GNDBB"
- note added: "Isolated valve driver + Power jack"
- note added: "MCU (Teensy 3.6) + RS485 converters + DC/DC converters for module power"
- note added: "NOTE: This design file is part of the Sanworks Bpod-CAD repository. (C) 2017 Sanworks LLC"
- note added: "Please read GPL v3.0 for license terms. http//www.gnu.org/licenses/gpl-3.0.en.html"
- note added: "Port1In"
- note added: "Port1LED"
- note added: "Port2In"
- note added: "Port2LED"
- note added: "Port3In"
- note added: "Port3LED"
- note added: "Port4In"
- note added: "Port4LED"
- note added: "RGB Status LED"
- note added: "Sanworks LLC"
- note added: "VLV1in"
- note added: "VLV1out"
- note added: "VLV2in"
- note added: "VLV2out"
- note added: "VLV3in"
- note added: "VLV3out"
- note added: "VLV4in"
- note added: "VLV4out"
- note added: "http://github.com/sanworks/Bpod-CAD"
- moved on the sheet: C1, C10, C2, C3, C4, C5, C6, C7, C8, C9, F1, IC1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
